Commit message: simulation

File: Rizon4r_with_kendama.urdf (robot description, URDF)
Before this commit: robot rizon4r, 28 links, 27 joints
Joints:
- removed joint kendama_to_ball
- removed joint kendama_to_string_1
- removed joint string_1_to_string_2
- removed joint string_2_to_string_3
- removed joint string_3_to_string_4
- removed joint string_4_to_string_5
- removed joint string_5_to_string_6
- removed joint string_6_to_string_7
- removed joint string_7_to_string_8
- joint joint1: origin xyz=0.0 0.0 0.155 rpy=0.0 0.0 -3.141592653589793 -> xyz=0.0 0.0 0.155 rpy=0.0 0.0 0.0
- joint joint2: origin xyz=0.0 0.03 0.21 rpy=0.0 0.0 0.0 -> xyz=0.0 0.03 0.21 rpy=-1.57079632679 0 0
- joint joint3: origin xyz=0.0 0.035 0.205 rpy=0.0 0.0 0.0 -> xyz=0.0 0.035 0.205 rpy=1.57079632679 0 0
- joint joint4: origin xyz=-0.02 -0.03 0.19 rpy=0.0 0.0 -3.141592653589793 -> xyz=-0.02 -0.03 0.19 rpy=1.57079632679 0 0
- joint joint5: origin xyz=-0.02 0.025 0.195 rpy=0.0 0.0 -3.141592653589793 -> xyz=-0.02 0.025 0.195 rpy=-1.57079632679 0 0
- joint joint6: origin xyz=0.0 0.03 0.19 rpy=0.0 0.0 0.0 -> xyz=0.0 0.03 0.19 rpy=1.57079632679 0 0.0
- joint joint7: origin xyz=-0.015 0.073 0.11 rpy=0.0 -1.5707963478683205 0.0 -> xyz=-0.015 0.073 0.11 rpy=0.0 0 0.0
- joint kendama_to_big_cup: origin xyz=0.135 0.04 0.0 rpy=0.0 0.0 0.0 -> xyz=0.135 -0.04 0.0 rpy=0.0 0.0 0.0
- joint kendama_to_small_cup: origin xyz=0.135 -0.04 0.0 rpy=0.0 0.0 0.0 -> xyz=0.135 0.04 0.0 rpy=0.0 0.0 0.0

Commit message: successfully places ball on top of big cup

File: Rizon4r_with_kendama.urdf (robot description, URDF)
Before this commit: robot rizon4r, 28 links, 18 joints
Links:
- removed link kendama_ball
- removed link kendama_string_1
- removed link kendama_string_2
- removed link kendama_string_3
- removed link kendama_string_4
- removed link kendama_string_5
- removed link kendama_string_6
- removed link kendama_string_7
- removed link kendama_string_8
- link kendama_big_cup: geometry collision cylinder length=0.018 radius=0.03; visual cylinder length=0.018 radius=0.03

Commit message: update urdf

File: Rizon4r_with_kendama.urdf (robot description, URDF)
Before this commit: robot rizon4r, 19 links, 18 joints
Joints:
- joint joint2: origin xyz=0.0 0.03 0.21 rpy=-1.57079632679 0 0 -> xyz=0.0 0.03 0.21 rpy=0.0 0 0
- joint joint3: origin xyz=0.0 0.035 0.205 rpy=1.57079632679 0 0 -> xyz=0.0 0.035 0.205 rpy=0.0 0 0
- joint joint4: origin xyz=-0.02 -0.03 0.19 rpy=1.57079632679 0 0 -> xyz=-0.02 -0.03 0.19 rpy=0 -0.43 0
- joint joint5: origin xyz=-0.02 0.025 0.195 rpy=-1.57079632679 0 0 -> xyz=-0.02 0.025 0.195 rpy=0 0 0
- joint joint7: origin xyz=-0.015 0.073 0.11 rpy=0.0 0 0.0 -> xyz=-0.015 0.073 0.11 rpy=0.0 0.0 0.0
