Commit message: Adding parallel kendama ee catch; increased gain in joint 6

File: Rizon4r_with_kendama_parallel.urdf (robot description, URDF)
Before this commit: robot rizon4r, 27 links, 26 joints
Joints:
- joint end_effector_to_kendama: origin xyz=0.065 0.0 0.0 rpy=-1.57079632679 -1.57079632679 0.0 -> xyz=0.065 0.0 0.0 rpy=0.0 0.0 0.0
